File: ECU.kicad_sch (KiCad schematic)
At the start: 0 parts

Commit message: Add power supply design
Parts:
- added C1, C13, C14, C2, C7, C8: 10uF,50V, Capacitor_SMD:CP_Elec_6.3x5.7, symbol Device:C_Polarized_Small_US
- added C10, C15, C16, C3, C4, C9: 100nF,50V, Capacitor_SMD:C_0603_1608Metric, symbol Device:C_Small
- added C11, C12, C17, C18, C5, C6: 47uF,35V, Capacitor_SMD:CP_Elec_8x10.5, symbol Device:C_Polarized_Small_US
- added C19: 22uF,10V, Capacitor_SMD:CP_Elec_5x3.9, symbol Device:C_Polarized_Small_US
- added D1, D2, D3: ~, Diode_SMD:D_SMC, symbol Device:D_Schottky
- added L1, L2, L3: 47uH, Inductor_SMD:L_Bourns_SRR1210A, symbol Device:L
- added R1: 220K, Resistor_SMD:R_0603_1608Metric, symbol Device:R_Small_US
- added R2, R5, R8: 10K, Resistor_SMD:R_0603_1608Metric, symbol Device:R_Small_US
- added R3, R6, R9: 0-10K, Potentiometer_SMD:Potentiometer_Bourns_3214J_Horizontal, symbol Device:R_Variable_US
- added R4: 120K, Resistor_SMD:R_0603_1608Metric, symbol Device:R_Small_US
- added R7: 47K, Resistor_SMD:R_0603_1608Metric, symbol Device:R_Small_US
- added U1, U2, U3: LM2678, Package_TO_SOT_SMD:TO-263-7_TabPin4, symbol ECU:LM2678
- added U4: LM3940, Package_TO_SOT_SMD:SOT-223-3_TabPin2, symbol ECU:LM3940
Connections:
- new net: C4.2, D1.1 (K), L1.1, U1.1 (OUT)
- new net: R2.2, R3.1
- new net: C16.2, D3.1 (K), L3.1, U3.1 (OUT)
- new net: R8.2, R9.1
- new net: C10.2, D2.1 (K), L2.1, U2.1 (OUT)
- new net: C16.1, U3.3 (CB)
- new net: R7.2, R8.1, U3.6 (FB)
- new net: R1.2, R2.1, U1.6 (FB)
- new net: C4.1, U1.3 (CB)
- new net: C10.1, U2.3 (CB)
- new net: R5.2, R6.1
- new net: R4.2, R5.1, U2.6 (FB)
- new net +12V: C11.1, C12.1, L2.2, R4.1
- new net +24V: C5.1, C6.1, L1.2, R1.1
- new net +3V3: C19.1, U4.3 (OUT)
- new net +5V: C17.1, C18.1, L3.2, R7.1, U4.1 (IN)
- new net GND: C1.2, C11.2, C12.2, C13.2, C14.2, C15.2, C17.2, C18.2, C19.2, C2.2, C3.2, C5.2, C6.2, C7.2, C8.2, C9.2, D1.2 (A), D2.2 (A), D3.2 (A), R3.2, R6.2, R9.2, U1.4 (GND), U2.4 (GND), U3.4 (GND), U4.2 (GND)
- new net VCC: C1.1, C13.1, C14.1, C15.1, C2.1, C3.1, C7.1, C8.1, C9.1, U1.2 (IN), U2.2 (IN), U3.2 (IN)
- no-connect marks 0 -> 3
Other:
- note added: "General Design Notes: - All voltage and current ratings are minimums - All MLCCs are X7R unless otherwise noted"
- note added: "Nominal output 14.5~27.8V"
- note added: "Nominal output 4.1~6.9V"
- note added: "Nominal output 8.5~15.7V"
- note added: "POWER SUPPLY"
- note added: "Power Supply Design Notes: - Input capacitors Irms >1A - Schottky diode reverse voltage >40V, current >5A - Inductor continuous current >5A - Each unit 4A output max due to thermal constraints - 3.3V LDO input capacitor omitted due to proximity to 5V regulator output"
